File: shield/shield.sch (KiCad schematic (older format))
At the start: 26 parts, among them P8 CONN_20X2, P8 CONN_3X2, P9 CONN_20X2, P9 CONN_3X2, U1 7805

Commit message: OOOOHHH LOOONG PIANO
Parts:
- gave numbers to parts that had none: 1
- renumbered BATTERY to BATTERY1, BBB to BBB1, DYNAMIXEL to DYNAMIXEL1, HEAD to HEAD1, IMU to IMU1, IR to IR1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
Connections:
- net +12V: now also BATTERY1.1 (P1); no longer BATTERY1.2 (PM)
- net GND: now also BATTERY1.2 (PM); no longer BATTERY1.1 (P1)
Other:
- moved on the sheet: BATTERY1
