File: shield/shield.sch (KiCad schematic (older format))
At the start: 26 parts, among them K1 CONN_3, U1 7805

Commit message: masmemoria
Parts:
- removed BBB1: CONN_20, symbol CONN_20
- removed K1: CONN_3, symbol CONN_3
- U1: value 7805 -> UBEC
- renumbered IMU1 to SENSORS
Connections:
- net +5V: now also Pnueve1.6 (P6); no longer SENSORS.3 (P3)
- net at OpenCM3.3 (P3): now also Pnueve1.21 (P21)
- net at OpenCM3.5 (P5): no longer Pnueve1.21 (P21)
- net +3.3V: now reaches Pnueve1.3 (P3)
- net +3.3V: now also Pnueve1.4 (P4), SENSORS.3 (P3)
Other:
- note added: "2"
- note added: "PLACA DE EXPASION PARA EL ROBOT RAIDER\n"
- moved on the sheet: BATTERY1, C1, C2, Pocho1, Pocho2, SENSORS, U1, proto1, proto2
